Commit message: Campaign C: forward walking with anatomical foot geometry (size 36)
654 support events, 120 s, forward on three MuJoCo builds (+2.49/+2.62/+2.58 m at roll -0.035; measured maximum +9.695622 m at roll -0.05 on 3.11.0). Foot corrected from 29.5 cm to 22.5 cm; centre of pressure identified as the variable governing direction. Five of six gait criteria met. Canon updated: jump, envelope, load, heels. T18 retracted. Outside the roll plateau the direction alternates with solver and numpy build (declared in README).

File: models/tx34_piedevero.urdf (robot description, URDF)
Before this commit: robot TX34_NOVA, 27 links, 26 joints
Links:
- link l_foot: geometry collision box size=0.1700 0.0900 0.0400; visual box size=0.1700 0.0900 0.0400
- link l_toe: geometry collision box size=0.0500 0.0900 0.0360; visual box size=0.0500 0.0900 0.0360
- link r_foot: geometry collision box size=0.1700 0.0900 0.0400; visual box size=0.1700 0.0900 0.0400
- link r_toe: geometry collision box size=0.0500 0.0900 0.0360; visual box size=0.0500 0.0900 0.0360
Joints:
- joint l_ankle_roll: limit lower=-0.2300 upper=0.2300 effort=40.0 velocity=10.0 -> lower=-0.2300 upper=0.2300 effort=80.0 velocity=10.0
- joint l_elbow: limit lower=-2.3000 upper=0.0000 effort=8.0 velocity=10.0 -> lower=-2.3000 upper=0.0000 effort=30.0 velocity=10.0
- joint l_toe_pitch: origin xyz=0.16000 0.00000 -0.05000 rpy=0 0 0 -> xyz=0.11500 0.00000 -0.05000 rpy=0 0 0
- joint l_wrist_pitch: limit lower=-0.8000 upper=0.8000 effort=1.4 velocity=10.0 -> lower=-0.8000 upper=0.8000 effort=10.0 velocity=10.0
- joint r_ankle_roll: limit lower=-0.2300 upper=0.2300 effort=40.0 velocity=10.0 -> lower=-0.2300 upper=0.2300 effort=80.0 velocity=10.0
- joint r_elbow: limit lower=-2.3000 upper=0.0000 effort=8.0 velocity=10.0 -> lower=-2.3000 upper=0.0000 effort=30.0 velocity=10.0
- joint r_toe_pitch: origin xyz=0.16000 0.00000 -0.05000 rpy=0 0 0 -> xyz=0.11500 0.00000 -0.05000 rpy=0 0 0
- joint r_wrist_pitch: limit lower=-0.8000 upper=0.8000 effort=1.4 velocity=10.0 -> lower=-0.8000 upper=0.8000 effort=10.0 velocity=10.0
- joint waist_yaw: limit lower=-0.2793 upper=0.2793 effort=2.5 velocity=10.0 -> lower=-0.2793 upper=0.2793 effort=30.0 velocity=10.0
